File: xlx_dl_cable.sch (KiCad schematic (older format))
At the start: 0 parts

Commit message: add cpu and cpld, and a bit things
Parts:
- added C?: C, symbol C
- added C? (x2): 10pF, symbol C
- added R?: R, symbol R
- added U?: XC2C256-VQ100, symbol XC2C256-VQ100
- added U?: 24CXX, symbol 24CXX
- added U?: CY7C68013-100TQFP_0, cypress-fx2-TQFP-100, symbol CY7C68013-100TQFP_0
- added X?: CRYSTAL, symbol CRYSTAL
Connections:
- net labels added: +3.3V, CPLD_CLK, GND, POR, USB_DM, USB_DP, XTAL_IN, XTAL_OUT
- wire segments 0 -> 40

Commit message: backup
Parts:
- added R? (x7): 10K, symbol R
Connections:
- net labels added: SCL, SDA
- wire segments 40 -> 68
Changed lines of the file:
@@
-EESchema Schematic File Version 2  date 24/11/2011 14:54:36
+EESchema Schematic File Version 2  date 24/11/2011 21:11:00
 LIBS:power
 LIBS:device
@@
 Comment4 ""
 $EndDescr
+Wire Wire Line
+	2350 5200 2200 5200
+Wire Wire Line
+	6500 7850 6400 7850
+Wire Wire Line
+	5850 7850 5900 7850
+Connection ~ 6650 7100
+Wire Wire Line
+	6400 7100 6650 7100
+Wire Wire Line
+	6650 7000 6650 7200
+Wire Wire Line
+	6650 7200 6400 7200
+Wire Wire Line
+	1700 4950 1650 4950
+Wire Wire Line
+	5850 7200 5900 7200
+Wire Wire Line
+	5850 7000 5900 7000
+Connection ~ 8750 10650
+Wire Wire Line
+	8750 10850 8850 10850
+Wire Wire Line
+	8750 10650 8850 10650
+Wire Wire Line
+	8850 10450 8750 10450
+Wire Wire Line
+	10300 10350 10300 10450
+Wire Wire Line
+	10300 10450 10250 10450
+Wire Wire Line
+	10250 10750 10650 10750
+Wire Wire Line
+	2350 4600 1700 4600
+Connection ~ 2250 7900
+Wire Wire Line
+	2250 7900 2350 7900
+Wire Wire Line
+	2350 3850 1700 3850
+Wire Wire Line
+	2350 4100 1700 4100
+Wire Wire Line
+	5700 10750 6300 10750
+Wire Wire Line
+	5150 10450 5300 10450
+Connection ~ 5300 10450
+Connection ~ 5800 10750
+Connection ~ 5800 10150
+Wire Wire Line
+	6300 10150 5700 10150
+Wire Wire Line
+	7800 9850 7800 9900
+Wire Wire Line
+	7800 11000 7800 10900
+Wire Wire Line
+	2350 6800 2250 6800
+Connection ~ 2250 7000
+Wire Wire Line
+	2250 7000 2350 7000
+Connection ~ 2250 7200
+Wire Wire Line
+	2250 7200 2350 7200
+Connection ~ 2250 7400
+Wire Wire Line
+	2250 7400 2350 7400
+Connection ~ 2250 7600
+Wire Wire Line
+	2250 7600 2350 7600
+Connection ~ 2250 3600
+Wire Wire Line
+	2350 3600 2250 3600
+Connection ~ 2250 3400
+Wire Wire Line
+	2250 3400 2350 3400
+Connection ~ 2250 3200
+Wire Wire Line
+	2250 3200 2350 3200
+Connection ~ 2250 3000
+Wire Wire Line
+	2250 3000 2350 3000
+Connection ~ 2250 2800
+Wire Wire Line
+	2250 2800 2350 2800
+Wire Wire Line
+	2350 3700 2250 3700
+Wire Wire Line
+	2250 2700 2350 2700
+Wire Wire Line
+	2250 2900 2350 2900
+Connection ~ 2250 2900
+Wire Wire Line
+	2250 3100 2350 3100
+Connection ~ 2250 3100
+Wire Wire Line
+	2250 3300 2350 3300
+Connection ~ 2250 3300
+Wire Wire Line
+	2250 3500 2350 3500
+Connection ~ 2250 3500
+Wire Wire Line
+	2250 3700 2250 2450
+Connection ~ 2250 2700
+Wire Wire Line
+	2250 7700 2350 7700
+Connection ~ 2250 7700
+Wire Wire Line
+	2250 7500 2350 7500
+Connection ~ 2250 7500
+Wire Wire Line
+	2250 7300 2350 7300
+Connection ~ 2250 7300
+Wire Wire Line
+	2250 7100 2350 7100
+Connection ~ 2250 7100
+Wire Wire Line
+	2350 6900 2250 6900
+Connection ~ 2250 6900
+Wire Wire Line
+	2250 6800 2250 8050
+Wire Wire Line
+	2250 7800 2350 7800
+Connection ~ 2250 7800
+Wire Wire Line
+	7800 10500 7800 10400
+Wire Wire Line
+	7200 10450 7800 10450
+Connection ~ 7800 10450
+Wire Wire Line
+	1700 4350 2350 4350
+Wire Wire Line
+	5300 10150 5300 10750
+Wire Wire Line
+	2350 4200 1700 4200
+Wire Wire Line
+	2350 3950 1700 3950
+Wire Wire Line
+	2350 6000 1700 6000
+Wire Wire Line
+	8700 5500 8000 5500
+Wire Wire Line
+	6850 7300 5850 7300
+Wire Wire Line
+	2350 4700 1700 4700
+Wire Wire Line
+	10250 10850 10650 10850
+Wire Wire Line
+	10400 10550 10250 10550
+Wire Wire Line
+	8850 10550 8750 10550
+Connection ~ 8750 10550
+Wire Wire Line
+	8750 10450 8750 10900
+Connection ~ 8750 10850
+Wire Wire Line
+	5900 7100 5850 7100
+Wire Wire Line
+	1650 5200 1700 5200
+Wire Wire Line
+	6400 7000 6800 7000
+Connection ~ 6650 7000
+Wire Wire Line
+	5900 7950 5850 7950
+Wire Wire Line
+	6400 7950 6550 7950
+Wire Wire Line
+	2200 4950 2350 4950
+$Comp
+L +3.3V #PWR?
+U 1 1 4ECE4231
+P 6500 7850
+F 0 "#PWR?" H 6500 7810 30  0001 C CNN
+F 1 "+3.3V" V 6500 8000 30  0000 C CNN
+	1    6500 7850
+	0    1    1    0
+$EndComp
+$Comp
+L GND #PWR?
+U 1 1 4ECE4213
+P 6550 7950
+F 0 "#PWR?" H 6550 7950 30  0001 C CNN
+F 1 "GND" H 6550 7880 30  0001 C CNN
+	1    6550 7950
+	0    -1   -1   0
+$EndComp
+$Comp
+L GND #PWR?
+U 1 1 4ECE41F1
+P 6800 7000
+F 0 "#PWR?" H 6800 7000 30  0001 C CNN
+F 1 "GND" H 6800 6930 30  0001 C CNN
+	1    6800 7000
+	0    -1   -1   0
+$EndComp
+$Comp
+L GND #PWR?
+U 1 1 4ECE41E5
+P 1650 4950
+F 0 "#PWR?" H 1650 4950 30  0001 C CNN
+F 1 "GND" H 1650 4880 30  0001 C CNN
+	1    1650 4950
+	0    1    1    0
+$EndComp
+$Comp
+L GND #PWR?
+U 1 1 4ECE41E1
+P 1650 5200
+F 0 "#PWR?" H 1650 5200 30  0001 C CNN
+F 1 "GND" H 1650 5130 30  0001 C CNN
+	1    1650 5200
+	0    1    1    0
+$EndComp
+$Comp
+L R R?
+U 1 1 4ECE41A1
+P 1950 5200
+F 0 "R?" V 1900 5400 50  0000 C CNN
+F 1 "10K" V 1950 5200 50  0000 C CNN
+	1    1950 5200
+	0    1    1    0
+$EndComp
+$Comp
+L R R?
+U 1 1 4ECE419C
+P 1950 4950
+F 0 "R?" V 1900 5150 50  0000 C CNN
+F 1 "10K" V 1950 4950 50  0000 C CNN
+	1    1950 4950
+	0    1    1    0
+$EndComp
+$Comp
+L R R?
+U 1 1 4ECE4184
+P 6150 7950
+F 0 "R?" V 6100 8150 50  0000 C CNN
+F 1 "10K" V 6150 7950 50  0000 C CNN
+	1    6150 7950
+	0    1    1    0
+$EndComp
+$Comp
+L R R?
+U 1 1 4ECE4181
+P 6150 7850
+F 0 "R?" V 6100 8050 50  0000 C CNN
+F 1 "10K" V 6150 7850 50  0000 C CNN
+	1    6150 7850
+	0    1    1    0
+$EndComp
+$Comp
+L R R?
+U 1 1 4ECE4160
+P 6150 7000
+F 0 "R?" V 6100 7200 50  0000 C CNN
+F 1 "10K" V 6150 7000 50  0000 C CNN
+	1    6150 7000
+	0    1    1    0
+$EndComp
+$Comp
+L R R?
+U 1 1 4ECE415C
+P 6150 7100
+F 0 "R?" V 6100 7300 50  0000 C CNN
+F 1 "10K" V 6150 7100 50  0000 C CNN
+	1    6150 7100
+	0    1    1    0
+$EndComp
+$Comp
+L R R?
+U 1 1 4ECE411F
+P 6150 7200
+F 0 "R?" V 6100 7400 50  0000 C CNN
+F 1 "10K" V 6150 7200 50  0000 C CNN
+	1    6150 7200
+	0    1    1    0
+$EndComp
+$Comp
+L GND #PWR?
+U 1 1 4ECE3F2F
+P 8750 10900
+F 0 "#PWR?" H 8750 10900 30  0001 C CNN
+F 1 "GND" H 8750 10830 30  0001 C CNN
+	1    8750 10900
+	1    0    0    -1
+$EndComp
+$Comp
+L GND #PWR?
+U 1 1 4ECE3F1E
+P 10400 10550
+F 0 "#PWR?" H 10400 10550 30  0001 C CNN
+F 1 "GND" H 10400 10480 30  0001 C CNN
+	1    10400 10550
+	0    -1   -1   0
+$EndComp
+$Comp
+L +3.3V #PWR?
+U 1 1 4ECE3E20
+P 10300 10350
+F 0 "#PWR?" H 10300 10310 30  0001 C CNN
+F 1 "+3.3V" H 10300 10460 30  0000 C CNN
+	1    10300 10350
+	1    0    0    -1
+$EndComp
+Text Label 10400 10850 0    60   ~ 0
+SDA
+Text Label 10400 10750 0    60   ~ 0
+SCL
+Text Label 1800 4700 0    60   ~ 0
+SDA
+Text Label 1800 4600 0    60   ~ 0
+SCL
+Text Label 6350 7300 0    60   ~ 0
+CPLD_CLK
 Text Label 8150 5500 0    60   ~ 0
 CPLD_CLK
-Wire Wire Line
-	8700 5500 8000 5500
-Wire Wire Line
-	2350 6000 1700 6000
-Wire Wire Line
-	2350 3950 1700 3950
-Wire Wire Line
-	2350 4200 1700 4200
-Wire Wire Line
-	5300 10750 5300 10150
-Wire Wire Line
-	1700 4350 2350 4350
-Connection ~ 7800 10450
-Wire Wire Line
-	7200 10450 7800 10450
-Wire Wire Line
-	7800 10400 7800 10500
-Connection ~ 2250 7800
-Wire Wire Line
-	2250 7800 2350 7800
-Wire Wire Line
-	2250 8050 2250 6800
-Connection ~ 2250 6900
-Wire Wire Line
-	2350 6900 2250 6900
-Connection ~ 2250 7100
-Wire Wire Line
-	2250 7100 2350 7100
-Connection ~ 2250 7300
-Wire Wire Line
-	2250 7300 2350 7300
-Connection ~ 2250 7500
-Wire Wire Line
-	2250 7500 2350 7500
-Connection ~ 2250 7700
-Wire Wire Line
-	2250 7700 2350 7700
-Connection ~ 2250 2700
-Wire Wire Line
-	2250 2450 2250 3700
-Connection ~ 2250 3500
-Wire Wire Line
-	2250 3500 2350 3500
-Connection ~ 2250 3300
-Wire Wire Line
-	2250 3300 2350 3300
-Connection ~ 2250 3100
-Wire Wire Line
-	2250 3100 2350 3100
-Connection ~ 2250 2900
-Wire Wire Line
-	2250 2900 2350 2900
-Wire Wire Line
-	2250 2700 2350 2700
-Wire Wire Line
-	2250 3700 2350 3700
-Wire Wire Line
-	2250 2800 2350 2800
-Connection ~ 2250 2800
-Wire Wire Line
-	2250 3000 2350 3000
-Connection ~ 2250 3000
-Wire Wire Line
-	2250 3200 2350 3200
-Connection ~ 2250 3200
-Wire Wire Line
-	2250 3400 2350 3400
-Connection ~ 2250 3400
-Wire Wire Line
-	2350 3600 2250 3600
-Connection ~ 2250 3600
-Wire Wire Line
-	2250 7600 2350 7600
-Connection ~ 2250 7600
-Wire Wire Line
-	2250 7400 2350 7400
-Connection ~ 2250 7400
-Wire Wire Line
-	2250 7200 2350 7200
-Connection ~ 2250 7200
-Wire Wire Line
-	2250 7000 2350 7000
-Connection ~ 2250 7000
-Wire Wire Line
-	2250 6800 2350 6800
-Wire Wire Line
-	7800 11000 7800 10900
-Wire Wire Line
-	7800 9850 7800 9900
-Wire Wire Line
-	5700 10150 6300 10150
-Connection ~ 5800 10150
-Connection ~ 5800 10750
-Connection ~ 5300 10450
-Wire Wire Line
-	5150 10450 5300 10450
-Wire Wire Line
-	6300 10750 5700 10750
-Wire Wire Line
-	2350 4100 1700 4100
-Wire Wire Line
-	2350 3850 1700 3850
-Wire Wire Line
-	2350 7900 2250 7900
-Connection ~ 2250 7900
 Text Label 1800 6000 0    60   ~ 0
 CPLD_CLK

Commit message: new part add, base finish
Parts:
- added C1, C10, C11, C12, C13, C16, C17, C18, C19, C2, C22, C23, C25, C27, C28, C29, C3, C30, C31, C4, C5, C7, C8, C9: 0.1uF, symbol C
- added C20, C24: 1uF, symbol C
- added C26: C, symbol C
- added C6: 3.3uF, symbol CP1
- added D1: LED_GREEN, symbol LED
- added D2: LED_RED, symbol LED
- added J1: USB_MINI_B, symbol USB_MINI_B
- added P1: CONN_8X2, symbol CONN_8X2
- added R1, R15, R16, R19, R2, R20, R21, R22, R23, R25, R26, R27, R28, R29, R3, R33, R34, R35, R36, R37, R4: 10K, symbol R
- added R17, R18: 2K, symbol R
- added R24: 10K/NP, symbol R
- added R30, R31, R32: 15R, symbol R
- added R7, R8: 0R, symbol R
- added U2: AMS1117-3.3V, symbol AMS1117
- added U4: AMS1117-1.8V, symbol AMS1117
- added U5: DS2411/NP, symbol DS2411
- added U7: 74HC244, symbol 74HC244
- C14, C15: renamed from C?; value 10pF -> 11pF
- C21: renamed from C?; value C -> 1uF
- R9: renamed from R?; value R -> 20K
- U6: renamed from U?; footprint (none) -> xilinx-VQ100
- X1: renamed from X?; value CRYSTAL -> 24MHz
- gave numbers to parts that had none: 9
Connections:
- net labels added: +1.8V, +5V, BIT_CLOCK, BUFFER_OE, COUNT0, COUNT1, COUNT2, COUNT3, COUNT4, CPLD_TCK, CPLD_TDI, CPLD_TDO, CPLD_TMS, CTRL2, CTRL3, GPIF_D00, GPIF_D01, GPIF_D02, GPIF_D03, GPIF_D04, GPIF_D05, GPIF_D06, GPIF_D07, GPIF_D08, GPIF_D09, GPIF_D10, GPIF_D11, GPIF_D12, GPIF_D13, GPIF_D14, GPIF_D15, GPIF_DONE, GPIF_START, JTAG_INIT, JTAG_TCK, JTAG_TD0, JTAG_TDI, JTAG_TMS, JTP_CMD0, JTP_CMD1, JTP_CMD2, JTP_CMD3, LAST_WORD, LED_GRN, LED_RED, RDY1, RDY2, SERIAL_NUMBER, SPARE_COM, TARGET_INIT, TARGET_TCK, TARGET_TD0, TARGET_TDI, TARGET_TMS, TARGET_VREF, TMS_LEVEL, VERSION_REQUEST, VREF_DETECT
- wire segments 68 -> 310
Other:
- note added: "Power"
- moved on the sheet: C14, C15, C21, R10, R11, R12, R13, R14, R5, R6, R9, U1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

Commit message: import to pcb file
Parts:
- C1, C10, C11, C12, C13, C14, C15, C16, C17, C18, C19, C2, C22, C23, C24, C25, C27, C28, C29, C3, C30, C31, C4, C5, C7, C8, C9: footprint (none) -> SM0603_Capa
- C20, C21, C6: footprint (none) -> SM0805
- C26: value C -> 0.1uF; footprint (none) -> SM0603_Capa
- D1, D2: footprint (none) -> LED-0805
- J1: footprint (none) -> USB_MINI_B
- P1: footprint (none) -> pin_array_8x2
- R1, R10, R11, R12, R13, R14, R15, R16, R17, R18, R19, R2, R20, R21, R22, R23, R24, R25, R26, R27, R28, R29, R3, R30, R31, R32, R33, R34, R35, R36, R37, R4, R5, R6, R7, R8, R9: footprint (none) -> SM0603
- U2, U4: footprint (none) -> SOT223
- U3: footprint (none) -> SO8N
- U5: footprint (none) -> SOT23_6
- U7: footprint (none) -> SO20L
- X1: footprint (none) -> HC-49V
Other:
- note added: "Core"
- note added: "Interface"
- note added: "LED"
- note added: "ROM"
- note added: "XTAL & Reset"
- note added: "miniUSB"
- moved on the sheet: C14, C15, X1

Commit message: backup
Connections:
- wire segments 310 -> 422
- no-connect marks 0 -> 51

Commit message: backup
Parts:
- C1, C10, C11, C12, C13, C14, C15, C16, C17, C18, C19, C2, C22, C23, C24, C25, C26, C27, C28, C29, C3, C30, C31, C4, C5, C7, C8, C9: footprint SM0603_Capa -> SM0603_0
- C20, C21, C6: footprint SM0805 -> SM0805_0
- D1, D2: footprint LED-0805 -> LED-0805_0
- J1: footprint USB_MINI_B -> Mini_USB_B_0
- R1, R10, R11, R12, R13, R14, R15, R16, R17, R18, R19, R2, R20, R21, R22, R23, R24, R25, R26, R27, R28, R29, R3, R30, R31, R32, R33, R34, R35, R36, R37, R4, R5, R6, R7, R8, R9: footprint SM0603 -> SM0603_0
- U5: footprint SOT23_6 -> SOT23_3_0
Connections:
- wire segments 422 -> 311
- no-connect marks 51 -> 48
Other:
- moved on the sheet: C30

Commit message: home work, base done
Parts:
- U7: footprint SO20L -> SSOP20
Changed lines of the file:
@@
-EESchema Schematic File Version 2  date 25/11/2011 17:38:19
+EESchema Schematic File Version 2  date 27/11/2011 12:14:28
 LIBS:power
 LIBS:device
@@
 LIBS:cypress-fx2
 LIBS:modify_from_lib
-LIBS:xlx_dl_cable-cache
 EELAYER 25  0
 EELAYER END
@@
 Sheet 1 1
 Title ""
-Date "25 nov 2011"
+Date "27 nov 2011"
 Rev ""
 Comp ""
@@
 F 0 "U7" H 12150 8700 60  0000 C CNN
 F 1 "74HC244" H 12200 7500 60  0000 C CNN
-F 2 "SO20L" H 12200 8100 60  0001 C CNN
+F 2 "SSOP20" H 12200 8100 60  0001 C CNN
 	1    12200 8100
 	1    0    0    -1
